File: Hardware/Punck_Components.kicad_sch (KiCad schematic)
At the start: 109 parts

Commit message: Component PCB Signal routing first draft
Parts:
- removed C31, C33, C35: (no value), symbol Device:C_Small
- removed C39: (no value), symbol Device:C_Polarized_Small
- removed D2: (no value), symbol Device:D_Schottky_Small
- removed J6: (no value), symbol Connector:USB_B_Micro
- removed TP10, TP11, TP12, TP9: (no value), symbol Connector:TestPoint
- removed U5: (no value), symbol Regulator_Switching:LM2675M-5
- added C1: 4.7uF, Capacitor_SMD:C_0603_1608Metric_Pad1.08x0.95mm_HandSolder, symbol Device:C_Small
- added C15, C18: 1uF, Capacitor_SMD:C_0603_1608Metric_Pad1.08x0.95mm_HandSolder, symbol Device:C_Small
- added C19: 100nF, Capacitor_SMD:C_0603_1608Metric_Pad1.08x0.95mm_HandSolder, symbol Device:C_Small
- added C36, C37: 10uF, Resistor_SMD:R_0805_2012Metric, symbol Device:C_Small
- added C39: 47uF, Resistor_SMD:R_1206_3216Metric, symbol Device:C_Small
- added R30: 33k, Resistor_SMD:R_0603_1608Metric_Pad0.98x0.95mm_HandSolder, symbol Device:R_Small
- added R31: 10k, Resistor_SMD:R_0603_1608Metric_Pad0.98x0.95mm_HandSolder, symbol Device:R_Small
- added R5: 100k, Resistor_SMD:R_0603_1608Metric, symbol Device:R_Small
- added U5: TPS561201, Package_TO_SOT_SMD:SOT-23-6_Handsoldering, symbol TPS561201:TPS561201
- C10, C11, C12, C13, C14, C2, C3, C4, C5, C6, C7, C8, C9: value (none) -> 100nF; footprint (none) -> Capacitor_SMD:C_0603_1608Metric_Pad1.08x0.95mm_HandSolder
- C16, C17: value (none) -> 2.2uF; footprint (none) -> Capacitor_SMD:C_0603_1608Metric_Pad1.08x0.95mm_HandSolder
- C20: renamed from C19; value (none) -> 30pF; footprint (none) -> Capacitor_SMD:C_0603_1608Metric_Pad1.08x0.95mm_HandSolder
- C21: value (none) -> 30pF; footprint (none) -> Capacitor_SMD:C_0603_1608Metric_Pad1.08x0.95mm_HandSolder
- C22: renamed from C1; value (none) -> 100pF; footprint (none) -> Capacitor_SMD:C_0603_1608Metric_Pad1.08x0.95mm_HandSolder
- C23: renamed from C15; value (none) -> 1nF; footprint (none) -> Capacitor_SMD:C_0603_1608Metric_Pad1.08x0.95mm_HandSolder
- C24: renamed from C18; value (none) -> 100pF; footprint (none) -> Capacitor_SMD:C_0603_1608Metric_Pad1.08x0.95mm_HandSolder
- C25: renamed from C20; value (none) -> 1nF; footprint (none) -> Capacitor_SMD:C_0603_1608Metric_Pad1.08x0.95mm_HandSolder
- C26: renamed from C22; value (none) -> 100nF; footprint (none) -> Capacitor_SMD:C_0603_1608Metric_Pad1.08x0.95mm_HandSolder
- C27: renamed from C23; value (none) -> 100nF; footprint (none) -> Capacitor_SMD:C_0603_1608Metric_Pad1.08x0.95mm_HandSolder
- C28: renamed from C24; value (none) -> 10uF; footprint (none) -> Capacitor_SMD:C_0805_2012Metric
- C29: renamed from C25; value (none) -> 100nF; footprint (none) -> Capacitor_SMD:C_0603_1608Metric_Pad1.08x0.95mm_HandSolder
- C30: renamed from C26; value (none) -> 10uF; footprint (none) -> Capacitor_SMD:C_0805_2012Metric
- C31: renamed from C27; value (none) -> 100nF; footprint (none) -> Capacitor_SMD:C_0603_1608Metric_Pad1.08x0.95mm_HandSolder
- C32: renamed from C28; value (none) -> 2.2uF; footprint (none) -> Capacitor_SMD:C_0603_1608Metric_Pad1.08x0.95mm_HandSolder
- C33: renamed from C29; value (none) -> 47uF; footprint (none) -> Capacitor_SMD:CP_Elec_5x5.8
- C34: value (none) -> 100nF; footprint (none) -> Resistor_SMD:R_0805_2012Metric; Part_Number (none) -> C57112
- C35: renamed from C30; value (none) -> 100nF; footprint (none) -> Capacitor_SMD:C_0603_1608Metric_Pad1.08x0.95mm_HandSolder
- C38: renamed from C32; value (none) -> 2.2uF; footprint (none) -> Capacitor_SMD:C_0603_1608Metric_Pad1.08x0.95mm_HandSolder
- C40: renamed from C36; value (none) -> 100nF; footprint (none) -> Capacitor_SMD:C_0603_1608Metric_Pad1.08x0.95mm_HandSolder
- C41: renamed from C37; value (none) -> 22uF; footprint (none) -> Capacitor_SMD:CP_Elec_4x5.8
- C42: renamed from C38; value (none) -> 2.2uF; footprint (none) -> Capacitor_SMD:C_0603_1608Metric_Pad1.08x0.95mm_HandSolder
- C44: renamed from C40; value (none) -> 22uF; footprint (none) -> Capacitor_SMD:CP_Elec_4x5.8
- D1: value (none) -> 1N5819; footprint (none) -> Diode_SMD:D_SOD-123
- D2: renamed from D3; value (none) -> 1N5819; footprint (none) -> Diode_SMD:D_SOD-123
- H1, H2: value (none) -> JLC_Tooling_Hole; footprint (none) -> Custom_Footprints:JLC_SMT_Tooling_Hole
- J1, J2, J3, J4: value (none) -> Conn_01x12_Female; footprint (none) -> Connector_PinHeader_2.54mm:PinHeader_1x12_P2.54mm_Vertical
- J5: value (none) -> SWD_Header; footprint (none) -> Custom_Footprints:SWD_header
- J7: value (none) -> Eurorack_10_pin_power; footprint (none) -> Custom_Footprints:Eurorack_10_pin_header
- L1: value (none) -> 3.3uH; footprint (none) -> Custom_Footprints:L_0806; Part_Number (none) -> C326343
- L2: value (none) -> L; footprint (none) -> Inductor_SMD:L_0805_2012Metric
- Q1, Q2, Q3, Q4, Q5, Q6, Q7: value (none) -> MMBT3904; footprint (none) -> Package_TO_SOT_SMD:SOT-23
- R1, R2: value (none) -> 4k7; footprint (none) -> Resistor_SMD:R_0603_1608Metric_Pad0.98x0.95mm_HandSolder
- R10: renamed from R17; value (none) -> 4k7; footprint (none) -> Resistor_SMD:R_0603_1608Metric_Pad0.98x0.95mm_HandSolder
- R11: renamed from R18; value (none) -> 4k7; footprint (none) -> Resistor_SMD:R_0603_1608Metric_Pad0.98x0.95mm_HandSolder
- R12: renamed from R3; value (none) -> 47k; footprint (none) -> Resistor_SMD:R_0603_1608Metric_Pad0.98x0.95mm_HandSolder
- R13: renamed from R6; value (none) -> 2k2; footprint (none) -> Resistor_SMD:R_0603_1608Metric_Pad0.98x0.95mm_HandSolder
- R14: renamed from R7; value (none) -> 10k; footprint (none) -> Resistor_SMD:R_0603_1608Metric_Pad0.98x0.95mm_HandSolder
- R15: renamed from R19; value (none) -> 4k7; footprint (none) -> Resistor_SMD:R_0603_1608Metric_Pad0.98x0.95mm_HandSolder
- R16: renamed from R8; value (none) -> 1k; footprint (none) -> Resistor_SMD:R_0603_1608Metric_Pad0.98x0.95mm_HandSolder
- R17: renamed from R20; value (none) -> 4k7; footprint (none) -> Resistor_SMD:R_0603_1608Metric_Pad0.98x0.95mm_HandSolder
- R18: renamed from R21; value (none) -> 4k7; footprint (none) -> Resistor_SMD:R_0603_1608Metric_Pad0.98x0.95mm_HandSolder
- R19: renamed from R22; value (none) -> 4k7; footprint (none) -> Resistor_SMD:R_0603_1608Metric_Pad0.98x0.95mm_HandSolder
- R20: renamed from R11; value (none) -> 47k; footprint (none) -> Resistor_SMD:R_0603_1608Metric_Pad0.98x0.95mm_HandSolder
- R21: renamed from R23; value (none) -> 1k; footprint (none) -> Resistor_SMD:R_0603_1608Metric_Pad0.98x0.95mm_HandSolder
- R22: renamed from R14; value (none) -> 2k2; footprint (none) -> Resistor_SMD:R_0603_1608Metric_Pad0.98x0.95mm_HandSolder
- R23: renamed from R15; value (none) -> 10k; footprint (none) -> Resistor_SMD:R_0603_1608Metric_Pad0.98x0.95mm_HandSolder
- R24: value (none) -> 1k; footprint (none) -> Resistor_SMD:R_0603_1608Metric_Pad0.98x0.95mm_HandSolder
- R25: renamed from R16; value (none) -> 1k; footprint (none) -> Resistor_SMD:R_0603_1608Metric_Pad0.98x0.95mm_HandSolder
- R26: renamed from R25; value (none) -> 1k; footprint (none) -> Resistor_SMD:R_0603_1608Metric_Pad0.98x0.95mm_HandSolder
- R27: renamed from R26; value (none) -> 1k; footprint (none) -> Resistor_SMD:R_0603_1608Metric_Pad0.98x0.95mm_HandSolder
- R28: renamed from R27; value (none) -> 1k; footprint (none) -> Resistor_SMD:R_0603_1608Metric_Pad0.98x0.95mm_HandSolder
- R29: renamed from R28; value (none) -> 1k; footprint (none) -> Resistor_SMD:R_0603_1608Metric_Pad0.98x0.95mm_HandSolder
- R3: renamed from R4; value (none) -> 4k7; footprint (none) -> Resistor_SMD:R_0603_1608Metric_Pad0.98x0.95mm_HandSolder
- R4: renamed from R5; value (none) -> 4k7; footprint (none) -> Resistor_SMD:R_0603_1608Metric_Pad0.98x0.95mm_HandSolder
- R6: renamed from R9; value (none) -> 4k7; footprint (none) -> Resistor_SMD:R_0603_1608Metric_Pad0.98x0.95mm_HandSolder
- R7: renamed from R10; value (none) -> 4k7; footprint (none) -> Resistor_SMD:R_0603_1608Metric_Pad0.98x0.95mm_HandSolder
- R8: renamed from R12; value (none) -> 4k7; footprint (none) -> Resistor_SMD:R_0603_1608Metric_Pad0.98x0.95mm_HandSolder
- R9: renamed from R13; value (none) -> 4k7; footprint (none) -> Resistor_SMD:R_0603_1608Metric_Pad0.98x0.95mm_HandSolder
- TP1, TP2, TP3, TP4, TP5: value (none) -> TestPoint; footprint (none) -> Custom_Footprints:1.3mm_Test_Point
- TP6, TP7, TP8: value (none) -> TestPoint; footprint (none) -> TestPoint:TestPoint_Pad_2.0x2.0mm
- U1: value (none) -> TL072; footprint (none) -> Package_SO:SOIC-8_3.9x4.9mm_P1.27mm
- U2: value (none) -> STM32H743ZITx; footprint (none) -> Package_QFP:LQFP-144_20x20mm_P0.5mm
- U3, U6: value (none) -> W25Q128JVS; footprint (none) -> Package_SO:SOIC-8_5.23x5.23mm_P1.27mm
- U4: value (none) -> PCM5100APW; footprint (none) -> Custom_Footprints:SSOP-20_4.4x6.5mm_Pitch0.65mm_Round_Pads
- U7: value (none) -> LD1117-3.3-4Tab; footprint (none) -> Package_TO_SOT_SMD:SOT-223-3_TabPin2
Connections:
- net QSPI_IO2 is gone; now on net QSPI_BK1_IO2: U2.1 (PE2)
- net SAMPLERA_IN is gone; now on net KICK_IN: J3.2 (Pin_2)
- net SAMPLERB_IN is gone; now on net OH_BTN: J4.2 (Pin_2)
- net +3.3VA: now also J3.12 (Pin_12), J4.12 (Pin_12), C15.2, C18.2, C19.2; no longer J1.1 (Pin_1), J4.1 (Pin_1)
- net +3V3: now also L1.2, C1.2, C39.1, R30.1; no longer L2.2, U7.2 (VO)
- net +5V: no longer L1.2, U7.3 (VI)
- net AUDIO_OUT_L: now also J4.10 (Pin_10); no longer J4.11 (Pin_11)
- net AUDIO_OUT_R: now also J4.11 (Pin_11); no longer J4.10 (Pin_10)
- net CH_BTN: now also J2.10 (Pin_10), U2.69 (PB10); no longer J1.7 (Pin_7), U2.13 (PF3)
- net CH_CLAMP: now also U2.128 (PG13); no longer U2.136 (PB6)
- net CH_IN: now also J3.6 (Pin_6); no longer J2.3 (Pin_3)
- net CH_LED: now also J4.8 (Pin_8); no longer J1.8 (Pin_8)
- net CH_LED_OUT: now also U2.97 (PC7); no longer U2.98 (PC8)
- net DAC_LRCLK: now also U2.73 (PB12); no longer U2.140 (PB9)
- net GND: now also J1.1 (Pin_1), J3.1 (Pin_1), J4.1 (Pin_1), C1.1, C15.1, C18.1, C19.1, C36.2, C37.2, C39.2, R31.2, R5.1, U5.1 (GND); no longer C34.2, J1.12 (Pin_12), J3.12 (Pin_12), J4.12 (Pin_12), U2.138 (BOOT0)
- net HIHAT_DECAY_POT: now also J1.12 (Pin_12); no longer J3.3 (Pin_3)
- net HIHAT_VOL_POT: now also J2.1 (Pin_1); no longer J3.4 (Pin_4)
- net KICK_ATTACK_POT: now also J1.4 (Pin_4); no longer J2.6 (Pin_6)
- net KICK_CLAMP: now also U2.141 (PE0); no longer U2.137 (PB7)
- net KICK_DECAY_POT: now also J1.5 (Pin_5); no longer J2.7 (Pin_7)
- net KICK_IN: no longer J1.2 (Pin_2)
- net KICK_VOL_POT: now also J1.6 (Pin_6); no longer J2.8 (Pin_8)
- net KI_BTN: now also J2.11 (Pin_11), U2.78 (PD9); no longer J2.1 (Pin_1), U2.10 (PF0)
- net KI_LED: now also J4.6 (Pin_6); no longer J2.2 (Pin_2)
- net KI_LED_OUT: now also U2.99 (PC9); no longer U2.96 (PC6)
- net MIDI_IN: now also J3.7 (Pin_7); no longer J4.6 (Pin_6)
- net MIDI_LEARN: now also J2.5 (Pin_5), U2.64 (PE11); no longer J4.7 (Pin_7), U2.67 (PE14)
- net OH_BTN: now also U2.114 (PD0); no longer J1.5 (Pin_5), U2.12 (PF2)
- net OH_CLAMP: now also U2.124 (PG9); no longer U2.93 (PG8)
- net OH_IN: now also J3.8 (Pin_8); no longer J3.1 (Pin_1)
- net OH_LED: now also J4.9 (Pin_9); no longer J1.6 (Pin_6)
- net OH_LED_OUT: now also U2.96 (PC6); no longer U2.99 (PC9)
- net SAMPLER_A_CLAMP: now also U2.137 (PB7); no longer U2.125 (PG10)
- net SAMPLER_A_IN: now also J3.3 (Pin_3)
- net SAMPLER_A_SPEED_POT: now also J1.3 (Pin_3); no longer J3.6 (Pin_6)
- net SAMPLER_A_VOICE_POT: now also J1.2 (Pin_2); no longer J3.5 (Pin_5)
- net SAMPLER_A_VOL_POT: now also J1.10 (Pin_10); no longer J3.7 (Pin_7)
- net SAMPLER_B_CLAMP: now also U2.135 (PB5); no longer U2.128 (PG13)
- net SAMPLER_B_IN: now also J3.5 (Pin_5)
- net SAMPLER_B_SPEED_POT: now also J2.2 (Pin_2); no longer J3.9 (Pin_9)
- net SAMPLER_B_VOICE_POT: now also J1.11 (Pin_11); no longer J3.8 (Pin_8)
- net SAMPLER_B_VOL_POT: now also J2.3 (Pin_3); no longer J3.10 (Pin_10)
- net SA_BTN: now also J2.7 (Pin_7), U2.66 (PE13); no longer J1.9 (Pin_9), U2.14 (PF4)
- net SA_LED: now also J3.10 (Pin_10); no longer J1.10 (Pin_10)
- net SB_BTN: now also J2.8 (Pin_8), U2.67 (PE14); no longer J2.4 (Pin_4), U2.15 (PF5)
- net SB_LED: now also J3.11 (Pin_11); no longer J2.5 (Pin_5)
- net SEQ_SELECT: now also J2.6 (Pin_6), U2.65 (PE12); no longer J4.8 (Pin_8), U2.68 (PE15)
- net SNARE_CLAMP: now also U2.136 (PB6); no longer U2.135 (PB5)
- net SNARE_FILTER_POT: now also J1.7 (Pin_7); no longer J2.9 (Pin_9)
- net SNARE_IN: now also J3.4 (Pin_4); no longer J1.11 (Pin_11)
- net SNARE_TUNING_POT: now also J1.8 (Pin_8); no longer J2.10 (Pin_10)
- net SNARE_VOL_POT: now also J1.9 (Pin_9); no longer J2.11 (Pin_11)
- net SN_BTN: now also J2.9 (Pin_9), U2.68 (PE15); no longer J1.3 (Pin_3), U2.11 (PF1)
- net SN_LED: now also J4.7 (Pin_7); no longer J1.4 (Pin_4)
- net SN_LED_OUT: now also U2.98 (PC8); no longer U2.97 (PC7)
- net TEMPO_OUT: now also J3.9 (Pin_9); no longer J3.11 (Pin_11)
- net TEMPO_POT: now also J2.4 (Pin_4); no longer J4.9 (Pin_9)
- net VCC: now also U7.3 (VI), C36.1, C37.1, U5.3 (VIN), U5.5 (EN); no longer C34.1
- net VSW: now also C34.1, U5.2 (SW)
- net MIDI_RX renamed MIDI_CLAMP
- net MIDI_CLAMP: now also U2.125 (PG10); no longer U2.141 (PE0)
- new net: R5.2, U2.138 (BOOT0)
- new net CB: C34.2, U5.6 (VBST)
- new net FB: R30.2, R31.1, U5.4 (VFB)
- new net VO: L2.2, U7.2 (VO)
- no-connect marks 57 -> 48
Other:
- note added: "FIXME Tempo out - amplifier Other Test connectors: DAC UART ADC MISC IO"
- note removed: "C54: 47uF 25V MLCC on Prototype"
- note removed: "Other Test connectors: DAC UART ADC MISC IO"
- note removed: "Tantalum"
- moved on the sheet: C14, C16, C17, C22, C23, C24, C25, C33, C44, L2, R12, R13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

Commit message: More component routing
Parts:
- removed U1: TL072, Package_SO:SOIC-8_3.9x4.9mm_P1.27mm, symbol Amplifier_Operational:TL072
- added R11, R8: (no value), symbol Device:R
- added R12: (no value), symbol Device:R_Small
- added U1: (no value), symbol Amplifier_Operational:TL074
- C1: value 4.7uF -> (none); footprint Capacitor_SMD:C_0603_1608Metric_Pad1.08x0.95mm_HandSolder -> (none)
- C10, C11, C12, C13, C14, C19, C2, C26, C27, C29, C3, C31, C35, C4, C40, C5, C6, C7, C8, C9: value 100nF -> (none); footprint Capacitor_SMD:C_0603_1608Metric_Pad1.08x0.95mm_HandSolder -> (none)
- C15, C18: value 1uF -> (none); footprint Capacitor_SMD:C_0603_1608Metric_Pad1.08x0.95mm_HandSolder -> (none)
- C16, C17, C32, C38, C42: value 2.2uF -> (none); footprint Capacitor_SMD:C_0603_1608Metric_Pad1.08x0.95mm_HandSolder -> (none)
- C20, C21: value 30pF -> (none); footprint Capacitor_SMD:C_0603_1608Metric_Pad1.08x0.95mm_HandSolder -> (none)
- C22, C24: value 100pF -> (none); footprint Capacitor_SMD:C_0603_1608Metric_Pad1.08x0.95mm_HandSolder -> (none)
- C23, C25: value 1nF -> (none); footprint Capacitor_SMD:C_0603_1608Metric_Pad1.08x0.95mm_HandSolder -> (none)
- C28, C30: value 10uF -> (none); footprint Capacitor_SMD:C_0805_2012Metric -> (none)
- C33: value 47uF -> (none); footprint Capacitor_SMD:CP_Elec_5x5.8 -> (none)
- C34: value 100nF -> (none); footprint Resistor_SMD:R_0805_2012Metric -> (none)
- C36, C37: value 10uF -> (none); footprint Resistor_SMD:R_0805_2012Metric -> (none)
- C39: value 47uF -> (none); footprint Resistor_SMD:R_1206_3216Metric -> (none)
- C41: value 22uF -> (none); footprint Capacitor_SMD:CP_Elec_4x5.8 -> (none)
- C43: renamed from C44; value 22uF -> (none); footprint Capacitor_SMD:CP_Elec_4x5.8 -> (none)
- D1, D2: value 1N5819 -> (none); footprint Diode_SMD:D_SOD-123 -> (none)
- H1, H2: value JLC_Tooling_Hole -> (none); footprint Custom_Footprints:JLC_SMT_Tooling_Hole -> (none)
- J1, J2, J3, J4: value Conn_01x12_Female -> (none); footprint Connector_PinHeader_2.54mm:PinHeader_1x12_P2.54mm_Vertical -> (none)
- J5: value SWD_Header -> (none); footprint Custom_Footprints:SWD_header -> (none)
- J6: renamed from J7; value Eurorack_10_pin_power -> (none); footprint Custom_Footprints:Eurorack_10_pin_header -> (none)
- L1: value 3.3uH -> (none); footprint Custom_Footprints:L_0806 -> (none)
- L2: value L -> (none); footprint Inductor_SMD:L_0805_2012Metric -> (none)
- Q1, Q2, Q3, Q4, Q5, Q6, Q7: value MMBT3904 -> (none); footprint Package_TO_SOT_SMD:SOT-23 -> (none)
- R1, R2, R3, R4, R6, R7: value 4k7 -> (none); footprint Resistor_SMD:R_0603_1608Metric_Pad0.98x0.95mm_HandSolder -> (none)
- R10: renamed from R9; value 4k7 -> (none); footprint Resistor_SMD:R_0603_1608Metric_Pad0.98x0.95mm_HandSolder -> (none)
- R13: renamed from R10; value 4k7 -> (none); footprint Resistor_SMD:R_0603_1608Metric_Pad0.98x0.95mm_HandSolder -> (none)
- R14: renamed from R11; value 4k7 -> (none); footprint Resistor_SMD:R_0603_1608Metric_Pad0.98x0.95mm_HandSolder -> (none)
- R15: renamed from R12; value 47k -> (none); footprint Resistor_SMD:R_0603_1608Metric_Pad0.98x0.95mm_HandSolder -> (none)
- R16: renamed from R13; value 2k2 -> (none); footprint Resistor_SMD:R_0603_1608Metric_Pad0.98x0.95mm_HandSolder -> (none)
- R17: renamed from R14; value 10k -> (none); footprint Resistor_SMD:R_0603_1608Metric_Pad0.98x0.95mm_HandSolder -> (none)
- R18: renamed from R15; value 4k7 -> (none); footprint Resistor_SMD:R_0603_1608Metric_Pad0.98x0.95mm_HandSolder -> (none)
- R19: renamed from R16; value 1k -> (none); footprint Resistor_SMD:R_0603_1608Metric_Pad0.98x0.95mm_HandSolder -> (none)
- R20: renamed from R17; value 4k7 -> (none); footprint Resistor_SMD:R_0603_1608Metric_Pad0.98x0.95mm_HandSolder -> (none)
- R21: renamed from R18; value 4k7 -> (none); footprint Resistor_SMD:R_0603_1608Metric_Pad0.98x0.95mm_HandSolder -> (none)
- R22: renamed from R19; value 4k7 -> (none); footprint Resistor_SMD:R_0603_1608Metric_Pad0.98x0.95mm_HandSolder -> (none)
- R23: renamed from R20; value 47k -> (none); footprint Resistor_SMD:R_0603_1608Metric_Pad0.98x0.95mm_HandSolder -> (none)
- R24: renamed from R21; value 1k -> (none); footprint Resistor_SMD:R_0603_1608Metric_Pad0.98x0.95mm_HandSolder -> (none)
- R25: renamed from R22; value 2k2 -> (none); footprint Resistor_SMD:R_0603_1608Metric_Pad0.98x0.95mm_HandSolder -> (none)
- R26: renamed from R23; value 10k -> (none); footprint Resistor_SMD:R_0603_1608Metric_Pad0.98x0.95mm_HandSolder -> (none)
- R27: renamed from R24; value 1k -> (none); footprint Resistor_SMD:R_0603_1608Metric_Pad0.98x0.95mm_HandSolder -> (none)
- R28: renamed from R25; value 1k -> (none); footprint Resistor_SMD:R_0603_1608Metric_Pad0.98x0.95mm_HandSolder -> (none)
- R29: renamed from R26; value 1k -> (none); footprint Resistor_SMD:R_0603_1608Metric_Pad0.98x0.95mm_HandSolder -> (none)
- R30: renamed from R27; value 1k -> (none); footprint Resistor_SMD:R_0603_1608Metric_Pad0.98x0.95mm_HandSolder -> (none)
- R31: renamed from R28; value 1k -> (none); footprint Resistor_SMD:R_0603_1608Metric_Pad0.98x0.95mm_HandSolder -> (none)
- R32: renamed from R29; value 1k -> (none); footprint Resistor_SMD:R_0603_1608Metric_Pad0.98x0.95mm_HandSolder -> (none)
- R33: renamed from R30; value 33k -> (none); footprint Resistor_SMD:R_0603_1608Metric_Pad0.98x0.95mm_HandSolder -> (none)
- R34: renamed from R31; value 10k -> (none); footprint Resistor_SMD:R_0603_1608Metric_Pad0.98x0.95mm_HandSolder -> (none)
- R5: value 100k -> (none); footprint Resistor_SMD:R_0603_1608Metric -> (none)
- R9: renamed from R8; value 4k7 -> (none); footprint Resistor_SMD:R_0603_1608Metric_Pad0.98x0.95mm_HandSolder -> (none)
- TP1, TP2, TP3, TP4, TP5: value TestPoint -> (none); footprint Custom_Footprints:1.3mm_Test_Point -> (none)
- TP6, TP7, TP8: value TestPoint -> (none); footprint TestPoint:TestPoint_Pad_2.0x2.0mm -> (none)
- U2: value STM32H743ZITx -> (none); footprint Package_QFP:LQFP-144_20x20mm_P0.5mm -> (none)
- U3, U6: value W25Q128JVS -> (none); footprint Package_SO:SOIC-8_5.23x5.23mm_P1.27mm -> (none)
- U4: value PCM5100APW -> (none); footprint Custom_Footprints:SSOP-20_4.4x6.5mm_Pitch0.65mm_Round_Pads -> (none)
- U5: value TPS561201 -> (none); footprint Package_TO_SOT_SMD:SOT-23-6_Handsoldering -> (none)
- U7: value LD1117-3.3-4Tab -> (none); footprint Package_TO_SOT_SMD:SOT-223-3_TabPin2 -> (none)
Connections:
- net +3.3VA: no longer J3.12 (Pin_12)
- net AUDIO_OUT_L: now also J4.9 (Pin_9); no longer J4.10 (Pin_10)
- net CH_LED: now also J4.7 (Pin_7); no longer J4.8 (Pin_8)
- net GND: now also R11.2, U1.10 (+), U1.12 (+), U1.5 (+)
- net KI_LED: now also J4.5 (Pin_5); no longer J4.6 (Pin_6)
- net OH_BTN: now also J3.11 (Pin_11); no longer J4.2 (Pin_2)
- net OH_LED: now also J4.8 (Pin_8); no longer J4.9 (Pin_9)
- net SA_LED: now also J3.9 (Pin_9); no longer J3.10 (Pin_10)
- net SB_LED: now also J3.10 (Pin_10); no longer J3.11 (Pin_11)
- net SN_LED: now also J4.6 (Pin_6); no longer J4.7 (Pin_7)
- net TEMPO_OUT: now also J4.10 (Pin_10), R12.2; no longer J3.9 (Pin_9), U2.134 (PB4)
- net USB_DM: now also J4.3 (Pin_3); no longer J4.4 (Pin_4)
- net USB_DP: now also J4.2 (Pin_2); no longer J4.3 (Pin_3)
- net USB_VBUS: now also J4.4 (Pin_4); no longer J4.5 (Pin_5)
- net VCC: now also U1.4 (V+)
- net VEE: now also U1.11 (V-)
- net TEMPO_CLOCK: now reaches U2.93 (PG8)
- net TEMPO_CLOCK: now also U1.3 (+)
- net at C22.1, R15.1, R19.1: now also U1.7
- net at C22.2, R15.2, R17.1: now also U1.6 (-)
- net at C24.2, R23.2, R26.1: now also U1.13 (-)
- net at C24.1, R23.1, R28.1: now also U1.14
- new net: R11.1, R8.2, U1.2 (-)
- new net: R12.1, R8.1, U1.1
- new net: U1.8, U1.9 (-)
- no-connect marks 48 -> 47
Other:
- moved on the sheet: C22, C23, R15, R16, R17, R19

Commit message: Component PCB first draft
Parts:
- added FID1: 4_Layer_Marker, Custom_Footprints:4_Layer_Markers, symbol Mechanical:Fiducial
- added J5: (no value), Connector_PinHeader_2.54mm:PinHeader_1x04_P2.54mm_Vertical, symbol Connector:Conn_01x04_Female
- added JP1: QSPI2_NCS_Select, Jumper:SolderJumper-3_P1.3mm_Bridged12_RoundedPad1.0x1.5mm, symbol Jumper:SolderJumper_3_Bridged12
- C1: renamed from C22; value (none) -> 100pF; footprint (none) -> Capacitor_SMD:C_0603_1608Metric_Pad1.08x0.95mm_HandSolder
- C10: renamed from C9; value (none) -> 100nF; footprint (none) -> Capacitor_SMD:C_0603_1608Metric_Pad1.08x0.95mm_HandSolder
- C11: renamed from C10; value (none) -> 100nF; footprint (none) -> Capacitor_SMD:C_0603_1608Metric_Pad1.08x0.95mm_HandSolder
- C12: renamed from C11; value (none) -> 100nF; footprint (none) -> Capacitor_SMD:C_0603_1608Metric_Pad1.08x0.95mm_HandSolder
- C13: renamed from C12; value (none) -> 100nF; footprint (none) -> Capacitor_SMD:C_0603_1608Metric_Pad1.08x0.95mm_HandSolder
- C14: renamed from C13; value (none) -> 100nF; footprint (none) -> Capacitor_SMD:C_0603_1608Metric_Pad1.08x0.95mm_HandSolder
- C15: renamed from C14; value (none) -> 100nF; footprint (none) -> Capacitor_SMD:C_0603_1608Metric_Pad1.08x0.95mm_HandSolder
- C16: renamed from C15; value (none) -> 1uF; footprint (none) -> Capacitor_SMD:C_0603_1608Metric_Pad1.08x0.95mm_HandSolder
- C17: renamed from C23; value (none) -> 2n2; footprint (none) -> Capacitor_SMD:C_0603_1608Metric_Pad1.08x0.95mm_HandSolder
- C18: renamed from C16; value (none) -> 2.2uF; footprint (none) -> Capacitor_SMD:C_0603_1608Metric_Pad1.08x0.95mm_HandSolder
- C19: renamed from C17; value (none) -> 2.2uF; footprint (none) -> Capacitor_SMD:C_0603_1608Metric_Pad1.08x0.95mm_HandSolder
- C2: renamed from C1; value (none) -> 4.7uF; footprint (none) -> Capacitor_SMD:C_0603_1608Metric_Pad1.08x0.95mm_HandSolder
- C20: renamed from C24; value (none) -> 100pF; footprint (none) -> Capacitor_SMD:C_0603_1608Metric_Pad1.08x0.95mm_HandSolder
- C21: renamed from C18; value (none) -> 1uF; footprint (none) -> Capacitor_SMD:C_0603_1608Metric_Pad1.08x0.95mm_HandSolder
- C22: renamed from C19; value (none) -> 100nF; footprint (none) -> Capacitor_SMD:C_0603_1608Metric_Pad1.08x0.95mm_HandSolder
- C23: renamed from C20; value (none) -> 30pF; footprint (none) -> Capacitor_SMD:C_0603_1608Metric_Pad1.08x0.95mm_HandSolder
- C24: renamed from C25; value (none) -> 2n2; footprint (none) -> Capacitor_SMD:C_0603_1608Metric_Pad1.08x0.95mm_HandSolder
- C25: renamed from C42; value (none) -> 2.2uF; footprint (none) -> Capacitor_SMD:C_0603_1608Metric_Pad1.08x0.95mm_HandSolder
- C26: renamed from C21; value (none) -> 30pF; footprint (none) -> Capacitor_SMD:C_0603_1608Metric_Pad1.08x0.95mm_HandSolder
- C27: renamed from C31; value (none) -> 100nF; footprint (none) -> Capacitor_SMD:C_0603_1608Metric_Pad1.08x0.95mm_HandSolder
- C28: renamed from C26; value (none) -> 100nF; footprint (none) -> Capacitor_SMD:C_0603_1608Metric_Pad1.08x0.95mm_HandSolder
- C29: renamed from C27; value (none) -> 100nF; footprint (none) -> Capacitor_SMD:C_0603_1608Metric_Pad1.08x0.95mm_HandSolder
- C3: renamed from C2; value (none) -> 100nF; footprint (none) -> Capacitor_SMD:C_0603_1608Metric_Pad1.08x0.95mm_HandSolder
- C30: renamed from C28; value (none) -> 10uF; footprint (none) -> Capacitor_SMD:C_0805_2012Metric
- C31: renamed from C29; value (none) -> 100nF; footprint (none) -> Capacitor_SMD:C_0603_1608Metric_Pad1.08x0.95mm_HandSolder
- C32: renamed from C30; value (none) -> 10uF; footprint (none) -> Capacitor_SMD:C_0805_2012Metric
- C33: renamed from C40; value (none) -> 100nF; footprint (none) -> Capacitor_SMD:C_0603_1608Metric_Pad1.08x0.95mm_HandSolder
- C34: renamed from C32; value (none) -> 2.2uF; footprint (none) -> Capacitor_SMD:C_0603_1608Metric_Pad1.08x0.95mm_HandSolder
- C35: value (none) -> 100nF; footprint (none) -> Capacitor_SMD:C_0603_1608Metric_Pad1.08x0.95mm_HandSolder
- C36: renamed from C38; value (none) -> 2.2uF; footprint (none) -> Capacitor_SMD:C_0603_1608Metric_Pad1.08x0.95mm_HandSolder
- C37: renamed from C33; value (none) -> 47uF; footprint (none) -> Capacitor_SMD:CP_Elec_5x5.8
- C38: renamed from C34; value (none) -> 100nF; footprint (none) -> Resistor_SMD:R_0805_2012Metric
- C39: renamed from C36; value (none) -> 10uF; footprint (none) -> Resistor_SMD:R_0805_2012Metric
- C4: renamed from C3; value (none) -> 100nF; footprint (none) -> Capacitor_SMD:C_0603_1608Metric_Pad1.08x0.95mm_HandSolder
- C40: renamed from C37; value (none) -> 10uF; footprint (none) -> Resistor_SMD:R_0805_2012Metric
- C41: renamed from C43; value (none) -> 22uF; footprint (none) -> Capacitor_SMD:CP_Elec_4x5.8
- C42: renamed from C39; value (none) -> 47uF; footprint (none) -> Resistor_SMD:R_1206_3216Metric
- C43: renamed from C41; value (none) -> 22uF; footprint (none) -> Capacitor_SMD:CP_Elec_4x5.8
- C5: renamed from C4; value (none) -> 100nF; footprint (none) -> Capacitor_SMD:C_0603_1608Metric_Pad1.08x0.95mm_HandSolder
- C6: renamed from C5; value (none) -> 100nF; footprint (none) -> Capacitor_SMD:C_0603_1608Metric_Pad1.08x0.95mm_HandSolder
- C7: renamed from C6; value (none) -> 100nF; footprint (none) -> Capacitor_SMD:C_0603_1608Metric_Pad1.08x0.95mm_HandSolder
- C8: renamed from C7; value (none) -> 100nF; footprint (none) -> Capacitor_SMD:C_0603_1608Metric_Pad1.08x0.95mm_HandSolder
- C9: renamed from C8; value (none) -> 100nF; footprint (none) -> Capacitor_SMD:C_0603_1608Metric_Pad1.08x0.95mm_HandSolder
- D1, D2: value (none) -> 1N5819; footprint (none) -> Diode_SMD:D_SOD-123
- H1, H2: value (none) -> JLC_Tooling_Hole; footprint (none) -> Custom_Footprints:JLC_SMT_Tooling_Hole
- J1, J2, J3, J4: value (none) -> Conn_01x12_Female; footprint (none) -> Connector_PinHeader_2.54mm:PinHeader_1x12_P2.54mm_Vertical
- J6: renamed from J5; value (none) -> SWD_Header; footprint (none) -> Custom_Footprints:SWD_header
- J7: renamed from J6; value (none) -> Eurorack_10_pin_power; footprint (none) -> Custom_Footprints:Eurorack_10_pin_header
- L1: value (none) -> 3.3uH; footprint (none) -> Custom_Footprints:L_0806
- L2: value (none) -> L; footprint (none) -> Inductor_SMD:L_0805_2012Metric
- Q1: renamed from Q6; value (none) -> MMBT3904; footprint (none) -> Package_TO_SOT_SMD:SOT-23
- Q2: renamed from Q3; value (none) -> MMBT3904; footprint (none) -> Package_TO_SOT_SMD:SOT-23
- Q3: renamed from Q1; value (none) -> MMBT3904; footprint (none) -> Package_TO_SOT_SMD:SOT-23
- Q4: renamed from Q5; value (none) -> MMBT3904; footprint (none) -> Package_TO_SOT_SMD:SOT-23
- Q5: renamed from Q7; value (none) -> MMBT3904; footprint (none) -> Package_TO_SOT_SMD:SOT-23
- Q6: renamed from Q2; value (none) -> MMBT3904; footprint (none) -> Package_TO_SOT_SMD:SOT-23
- Q7: renamed from Q4; value (none) -> MMBT3904; footprint (none) -> Package_TO_SOT_SMD:SOT-23
- R1: renamed from R18; value (none) -> 4k7; footprint (none) -> Resistor_SMD:R_0603_1608Metric_Pad0.98x0.95mm_HandSolder
- R10: renamed from R5; value (none) -> 100k; footprint (none) -> Resistor_SMD:R_0603_1608Metric
- R11: renamed from R6; value (none) -> 4k7; footprint (none) -> Resistor_SMD:R_0603_1608Metric_Pad0.98x0.95mm_HandSolder
- R12: renamed from R9; value (none) -> 4k7; footprint (none) -> Resistor_SMD:R_0603_1608Metric_Pad0.98x0.95mm_HandSolder
- R13: renamed from R23; value (none) -> 47k; footprint (none) -> Resistor_SMD:R_0603_1608Metric_Pad0.98x0.95mm_HandSolder
- R14: renamed from R25; value (none) -> 1k; footprint (none) -> Resistor_SMD:R_0603_1608Metric_Pad0.98x0.95mm_HandSolder
- R15: renamed from R26; value (none) -> 15k; footprint (none) -> Resistor_SMD:R_0603_1608Metric_Pad0.98x0.95mm_HandSolder
- R16: renamed from R28; value (none) -> 1k; footprint (none) -> Resistor_SMD:R_0603_1608Metric_Pad0.98x0.95mm_HandSolder
- R17: renamed from R1; value (none) -> 4k7; footprint (none) -> Resistor_SMD:R_0603_1608Metric_Pad0.98x0.95mm_HandSolder
- R18: renamed from R3; value (none) -> 4k7; footprint (none) -> Resistor_SMD:R_0603_1608Metric_Pad0.98x0.95mm_HandSolder
- R19: renamed from R24; value (none) -> 1k; footprint (none) -> Resistor_SMD:R_0603_1608Metric_Pad0.98x0.95mm_HandSolder
- R2: renamed from R15; value (none) -> 47k; footprint (none) -> Resistor_SMD:R_0603_1608Metric_Pad0.98x0.95mm_HandSolder
- R20: renamed from R13; value (none) -> 4k7; footprint (none) -> Resistor_SMD:R_0603_1608Metric_Pad0.98x0.95mm_HandSolder
- R21: renamed from R27; value (none) -> 1k; footprint (none) -> Resistor_SMD:R_0603_1608Metric_Pad0.98x0.95mm_HandSolder
- R22: renamed from R29; value (none) -> 1k; footprint (none) -> Resistor_SMD:R_0603_1608Metric_Pad0.98x0.95mm_HandSolder
- R23: renamed from R14; value (none) -> 4k7; footprint (none) -> Resistor_SMD:R_0603_1608Metric_Pad0.98x0.95mm_HandSolder
- R24: renamed from R30; value (none) -> 1k; footprint (none) -> Resistor_SMD:R_0603_1608Metric_Pad0.98x0.95mm_HandSolder
- R25: renamed from R31; value (none) -> 1k; footprint (none) -> Resistor_SMD:R_0603_1608Metric_Pad0.98x0.95mm_HandSolder
- R26: renamed from R32; value (none) -> 1k; footprint (none) -> Resistor_SMD:R_0603_1608Metric_Pad0.98x0.95mm_HandSolder
- R27: renamed from R20; value (none) -> 4k7; footprint (none) -> Resistor_SMD:R_0603_1608Metric_Pad0.98x0.95mm_HandSolder
- R28: renamed from R22; value (none) -> 4k7; footprint (none) -> Resistor_SMD:R_0603_1608Metric_Pad0.98x0.95mm_HandSolder
- R29: renamed from R2; value (none) -> 4k7; footprint (none) -> Resistor_SMD:R_0603_1608Metric_Pad0.98x0.95mm_HandSolder
- R3: renamed from R11; value (none) -> 10k; footprint (none) -> Resistor_SMD:R_0603_1608Metric_Pad0.98x0.95mm_HandSolder
- R30: renamed from R4; value (none) -> 4k7; footprint (none) -> Resistor_SMD:R_0603_1608Metric_Pad0.98x0.95mm_HandSolder
- R31: renamed from R7; value (none) -> 4k7; footprint (none) -> Resistor_SMD:R_0603_1608Metric_Pad0.98x0.95mm_HandSolder
- R32: renamed from R10; value (none) -> 4k7; footprint (none) -> Resistor_SMD:R_0603_1608Metric_Pad0.98x0.95mm_HandSolder
- R33: value (none) -> 33k; footprint (none) -> Resistor_SMD:R_0603_1608Metric_Pad0.98x0.95mm_HandSolder
- R34: value (none) -> 10k; footprint (none) -> Resistor_SMD:R_0603_1608Metric_Pad0.98x0.95mm_HandSolder
- R4: renamed from R8; value (none) -> 15k; footprint (none) -> Resistor_SMD:R_0603_1608Metric_Pad0.98x0.95mm_HandSolder
- R5: renamed from R21; value (none) -> 4k7; footprint (none) -> Resistor_SMD:R_0603_1608Metric_Pad0.98x0.95mm_HandSolder
- R6: renamed from R16; value (none) -> 1k; footprint (none) -> Resistor_SMD:R_0603_1608Metric_Pad0.98x0.95mm_HandSolder
- R7: renamed from R17; value (none) -> 15k; footprint (none) -> Resistor_SMD:R_0603_1608Metric_Pad0.98x0.95mm_HandSolder
- R8: renamed from R19; value (none) -> 1k; footprint (none) -> Resistor_SMD:R_0603_1608Metric_Pad0.98x0.95mm_HandSolder
- R9: renamed from R12; value (none) -> 1k; footprint (none) -> Resistor_SMD:R_0603_1608Metric_Pad0.98x0.95mm_HandSolder
- TP4: renamed from TP1; value (none) -> TestPoint; footprint (none) -> Custom_Footprints:1.3mm_Test_Point
- TP5: renamed from TP2; value (none) -> TestPoint; footprint (none) -> Custom_Footprints:1.3mm_Test_Point
- TP6: renamed from TP3; value (none) -> TestPoint; footprint (none) -> Custom_Footprints:1.3mm_Test_Point
- TP7: renamed from TP4; value (none) -> TestPoint; footprint (none) -> Custom_Footprints:1.3mm_Test_Point
- TP8: renamed from TP5; value (none) -> TestPoint; footprint (none) -> Custom_Footprints:1.3mm_Test_Point
- U1: value (none) -> TL074; footprint (none) -> Package_SO:SOIC-14_3.9x8.7mm_P1.27mm
- U2: value (none) -> STM32H743ZITx; footprint (none) -> Package_QFP:LQFP-144_20x20mm_P0.5mm
- U3: value (none) -> W25Q128JVS; footprint (none) -> Package_SO:SOIC-8_5.23x5.23mm_P1.27mm
- U4: value (none) -> PCM5100APW; footprint (none) -> Custom_Footprints:SSOP-20_4.4x6.5mm_Pitch0.65mm_Round_Pads
- U5: renamed from U6; value (none) -> W25Q128JVS; footprint (none) -> Package_SO:SOIC-8_5.23x5.23mm_P1.27mm
- U6: renamed from U5; value (none) -> TPS561201; footprint (none) -> Package_TO_SOT_SMD:SOT-23-6_Handsoldering
- U7: value (none) -> LD1117-3.3-4Tab; footprint (none) -> Package_TO_SOT_SMD:SOT-223-3_TabPin2
- Y1: value (none) -> 8MHz 20pF; footprint (none) -> Crystal:Crystal_SMD_5032-2Pin_5.0x3.2mm
- renumbered TP6 to TP1, TP7 to TP2, TP8 to TP3
Connections:
- net +3.3VA: now also R20.2, R27.2, R29.2, R31.2
- net +3V3: no longer R20.2, R27.2, R29.2, R31.2
- net CH_BTN: now also J2.4 (Pin_4), U2.64 (PE11); no longer J2.10 (Pin_10), U2.69 (PB10)
- net CH_CLAMP: now also U2.65 (PE12); no longer U2.128 (PG13)
- net CH_IN: now also J2.6 (Pin_6); no longer J3.6 (Pin_6)
- net DAC1: now also J5.2 (Pin_2)
- net DAC2: now also J5.1 (Pin_1)
- net GND: now also J3.12 (Pin_12)
- net HIHAT_DECAY_POT: now also J1.8 (Pin_8), U2.42 (PA6); no longer J1.12 (Pin_12), U2.46 (PB0)
- net KICK_CLAMP: now also Q2.3 (C), R11.1, U2.114 (PD0); no longer Q3.3 (C), R17.1, U2.141 (PE0)
- net KICK_IN: now also J3.11 (Pin_11), R12.1; no longer J3.2 (Pin_2), R18.1
- net KI_BTN: now also J3.3 (Pin_3), U2.136 (PB6); no longer J2.11 (Pin_11), U2.78 (PD9)
- net MIDI_IN: now also J3.9 (Pin_9); no longer J3.7 (Pin_7)
- net MIDI_LEARN: now also J2.10 (Pin_10), U2.69 (PB10); no longer J2.5 (Pin_5), U2.64 (PE11)
- net OH_BTN: now also J3.8 (Pin_8), U2.125 (PG10); no longer J3.11 (Pin_11), U2.114 (PD0)
- net OH_CLAMP: now also U2.66 (PE13); no longer U2.124 (PG9)
- net OH_IN: now also J2.7 (Pin_7); no longer J3.8 (Pin_8)
- net QSPI_BK2_NCS: now also JP1.1 (A); no longer U5.1 (~{CS})
- net SAMPLER_A_CLAMP: now also U2.67 (PE14); no longer U2.137 (PB7)
- net SAMPLER_A_IN: now also J2.8 (Pin_8); no longer J3.3 (Pin_3)
- net SAMPLER_A_SPEED_POT: now also J1.11 (Pin_11), U2.45 (PC5); no longer J1.3 (Pin_3), U2.27 (PC1)
- net SAMPLER_A_VOICE_POT: now also J1.3 (Pin_3), U2.27 (PC1); no longer J1.2 (Pin_2), U2.26 (PC0)
- net SAMPLER_A_VOL_POT: now also J2.2 (Pin_2), U2.49 (PF11); no longer J1.10 (Pin_10), U2.44 (PC4)
- net SAMPLER_B_CLAMP: now also U2.68 (PE15); no longer U2.135 (PB5)
- net SAMPLER_B_IN: now also J2.9 (Pin_9); no longer J3.5 (Pin_5)
- net SAMPLER_B_SPEED_POT: now also J1.9 (Pin_9), U2.43 (PA7); no longer J2.2 (Pin_2), U2.49 (PF11)
- net SAMPLER_B_VOICE_POT: now also J1.12 (Pin_12), U2.46 (PB0); no longer J1.11 (Pin_11), U2.45 (PC5)
- net SA_BTN: now also J3.2 (Pin_2), U2.137 (PB7); no longer J2.7 (Pin_7), U2.66 (PE13)
- net SA_LED: now also J3.5 (Pin_5); no longer J3.9 (Pin_9)
- net SB_BTN: now also J3.6 (Pin_6), U2.128 (PG13); no longer J2.8 (Pin_8), U2.67 (PE14)
- net SB_LED: now also J3.7 (Pin_7); no longer J3.10 (Pin_10)
- net SEQ_SELECT: now also J2.11 (Pin_11), U2.78 (PD9); no longer J2.6 (Pin_6), U2.65 (PE12)
- net SNARE_CLAMP: now also Q3.3 (C), R17.1, U2.124 (PG9); no longer Q2.3 (C), R11.1, U2.136 (PB6)
- net SNARE_FILTER_POT: now also J1.2 (Pin_2), U2.26 (PC0); no longer J1.7 (Pin_7), U2.37 (PA3)
- net SNARE_IN: now also J3.10 (Pin_10), R18.1; no longer J3.4 (Pin_4), R12.1
- net SNARE_TUNING_POT: now also J1.7 (Pin_7), U2.37 (PA3); no longer J1.8 (Pin_8), U2.42 (PA6)
- net SNARE_VOL_POT: now also J1.10 (Pin_10), U2.44 (PC4); no longer J1.9 (Pin_9), U2.43 (PA7)
- net SN_BTN: now also J3.4 (Pin_4), U2.135 (PB5); no longer J2.9 (Pin_9), U2.68 (PE15)
- net TEMPO_POT: now also J2.5 (Pin_5); no longer J2.4 (Pin_4)
- net OCTOSPIM_P2_NCS: now reaches U2.127 (PG12)
- net OCTOSPIM_P2_NCS: now also JP1.3 (B)
- net UART_RX: now reaches U2.18 (PF6)
- net UART_RX: now also J5.3 (Pin_3)
- net UART_TX: now reaches U2.19 (PF7)
- net UART_TX: now also J5.4 (Pin_4)
- net MIDI_CLAMP renamed MIDI_UART
- net MIDI_UART: now also U2.141 (PE0); no longer U2.125 (PG10)
- new net: JP1.2 (C), U5.1 (~{CS})
- no-connect marks 47 -> 51
Other:
- note added: "Analog 3.3V Supply"
- note added: "Connectors"
- note added: "DAC"
- note added: "Digital 3.3V Supply"
- note added: "Gain: -47k/16k = -2.94 Cutoff: 1 / (2π * 1000 * 2.2e-9) = 72kHz"
- note added: "Output Amplifiers"
- note removed: "FIXME Tempo out - amplifier Other Test connectors: DAC UART ADC MISC IO"
- note removed: "Headers and Connectors"
- note removed: "Output Amplifiers and Buffers"
- note removed: "Wet Output Amplifiers"
- moved on the sheet: C1, C10, C11, C12, C13, C14, C15, C16, C17, C2, C20, C24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
