File: Hardware/Punck_Components.kicad_sch (KiCad schematic)
At the start: 115 parts, among them J1 Conn_01x12_Female, J2 Conn_01x12_Female, J3 Conn_01x12_Female, J4 Conn_01x12_Female, J5 Debug_Header, J6 SWD_Header, J7 Eurorack_10_pin_power, Q1 MMBT3904, Q2 MMBT3904, Q3 MMBT3904, Q4 MMBT3904, Q5 MMBT3904, Q6 MMBT3904, Q7 MMBT3904, U1 TL074, U2 STM32H743ZITx, U3 W25Q128JVS, U4 PCM5100APW, U5 W25Q128JVS, U6 TPS561201, U7 LD1117-3.3-4Tab, Y1 8MHz 20pF

Commit message: Fixed incorrect pinout on transistors
Parts:
- Q1, Q2, Q3, Q4, Q5, Q6, Q7: symbol Transistor_BJT:2N3904 -> Transistor_BJT:MMBT3904
- R3: value 10k -> 15k
- R4: value 15k -> 10k
Connections:
- net GND: now also Q1.2 (E), Q2.2 (E), Q3.2 (E), Q4.2 (E), Q5.2 (E), Q6.2 (E), Q7.2 (E); no longer Q1.1 (E), Q2.1 (E), Q3.1 (E), Q4.1 (E), Q5.1 (E), Q6.1 (E), Q7.1 (E)
- net at R27.2: now also Q5.1 (B); no longer Q5.2 (B)
- net at R12.2: now also Q2.1 (B); no longer Q2.2 (B)
- net at R23.2: now also Q4.1 (B); no longer Q4.2 (B)
- net at R29.2: now also Q6.1 (B); no longer Q6.2 (B)
- net at R18.2: now also Q3.1 (B); no longer Q3.2 (B)
- net at R31.2: now also Q7.1 (B); no longer Q7.2 (B)
- net at R5.2: now also Q1.1 (B); no longer Q1.2 (B)
Other:
- note added: "Gain: 1 + 10k/15k = 1.66 Vout = 3.3 * 1.66 = 5.5V"
Changed lines of the file:
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@@
     (effects (font (size 1.27 1.27)) (justify left bottom))
   )
+  (text "Gain: 1 + 10k/15k = 1.66\nVout = 3.3 * 1.66 = 5.5V" (at 303.53 58.42 0)
+    (effects (font (size 1.27 1.27)) (justify left bottom))
+  )
   (text "ADC Pins\n--------\nPA0 ADC1_INP16       \nPA1 ADC1_INP17       \nPA2 ADC12_INP14      \nPA3 ADC12_INP15      \n[PA4 ADC12_INP18 DAC]\n[PA5 ADC12_INP19 DAC]\nPA6 ADC12_INP3       \nPA7 ADC12_INP7       \n                     \nPB0 ADC12_INP9       \nPB1 ADC12_INP5       \n                     \nPC0 ADC123_INP10     \nPC1 ADC123_INP11     \nPC2 ADC123_INP12     \n[PC3_C ADC3_INP1]    \nPC4 ADC12_INP4       \nPC5 ADC12_INP8       \n                     \nPF11 ADC1_INP2       \nPF12 ADC1_INP6       \nPF13 ADC2_INP2       \nPF14 ADC2_INP6       "
     (at -55.88 85.09 0)
@@
   )
   (symbol (lib_id "power:GND") (at 22.86 90.17 0) (unit 1)
-    (in_bom yes) (on_board yes)
+    (in_bom yes) (on_board yes) (fields_autoplaced)
     (property "Reference" "#PWR023" (id 0) (at 22.86 96.52 0)
       (effects (font (size 1.27 1.27)) hide)
     )
-    (property "Value" "GND" (id 1) (at 22.987 93.4212 90)
-      (effects (font (size 1.27 1.27)) (justify right))
-    )
+    (property "Value" "GND" (id 1) (at 22.86 95.25 0))
     (property "Footprint" "" (id 2) (at 22.86 90.17 0)
       (effects (font (size 1.27 1.27)) hide)
@@
     (in_bom yes) (on_board yes)
     (property "Reference" "R3" (id 0) (at 303.53 34.29 90))
-    (property "Value" "10k" (id 1) (at 303.53 31.75 90))
+    (property "Value" "15k" (id 1) (at 303.53 31.75 90))
     (property "Footprint" "Resistor_SMD:R_0603_1608Metric_Pad0.98x0.95mm_HandSolder" (id 2) (at 303.53 33.528 90)
       (effects (font (size 1.27 1.27)) hide)
@@
     (pin "4")
   )
-  (symbol (lib_id "Transistor_BJT:2N3904") (at 378.46 68.58 0) (unit 1)
+  (symbol (lib_id "Transistor_BJT:MMBT3904") (at 378.46 68.58 0) (unit 1)
     (in_bom yes) (on_board yes) (fields_autoplaced)
     (property "Reference" "Q2" (id 0) (at 383.54 67.3099 0)
@@
     (pin "2")
   )
-  (symbol (lib_id "Transistor_BJT:2N3904") (at 378.46 167.64 0) (unit 1)
+  (symbol (lib_id "Transistor_BJT:MMBT3904") (at 378.46 167.64 0) (unit 1)
     (in_bom yes) (on_board yes) (fields_autoplaced)
     (property "Reference" "Q5" (id 0) (at 383.54 166.3699 0)
@@
     (pin "2")
   )
-  (symbol (lib_id "Transistor_BJT:2N3904") (at 378.46 200.66 0) (unit 1)
+  (symbol (lib_id "Transistor_BJT:MMBT3904") (at 378.46 200.66 0) (unit 1)
     (in_bom yes) (on_board yes) (fields_autoplaced)
     (property "Reference" "Q6" (id 0) (at 383.54 199.3899 0)
@@
     (pin "2")
   )
-  (symbol (lib_id "Transistor_BJT:2N3904") (at 378.46 134.62 0) (unit 1)
+  (symbol (lib_id "Transistor_BJT:MMBT3904") (at 378.46 134.62 0) (unit 1)
     (in_bom yes) (on_board yes) (fields_autoplaced)
     (property "Reference" "Q4" (id 0) (at 383.54 133.3499 0)
@@
     (pin "1")
   )
-  (symbol (lib_id "Transistor_BJT:2N3904") (at 378.46 233.68 0) (unit 1)
+  (symbol (lib_id "Transistor_BJT:MMBT3904") (at 378.46 233.68 0) (unit 1)
     (in_bom yes) (on_board yes) (fields_autoplaced)
     (property "Reference" "Q7" (id 0) (at 383.54 232.4099 0)
@@
     (pin "1")
   )
-  (symbol (lib_id "Transistor_BJT:2N3904") (at 378.46 36.83 0) (unit 1)
+  (symbol (lib_id "Transistor_BJT:MMBT3904") (at 378.46 36.83 0) (unit 1)
     (in_bom yes) (on_board yes) (fields_autoplaced)
     (property "Reference" "Q1" (id 0) (at 383.54 35.5599 0)
@@
     (pin "1")
   )
-  (symbol (lib_id "Transistor_BJT:2N3904") (at 378.46 100.33 0) (unit 1)
+  (symbol (lib_id "Transistor_BJT:MMBT3904") (at 378.46 100.33 0) (unit 1)
     (in_bom yes) (on_board yes) (fields_autoplaced)
     (property "Reference" "Q3" (id 0) (at 383.54 99.0599 0)
@@
     (in_bom yes) (on_board yes)
     (property "Reference" "R4" (id 0) (at 316.23 34.29 90))
-    (property "Value" "15k" (id 1) (at 316.23 31.75 90))
+    (property "Value" "10k" (id 1) (at 316.23 31.75 90))
     (property "Footprint" "Resistor_SMD:R_0603_1608Metric_Pad0.98x0.95mm_HandSolder" (id 2) (at 316.23 33.528 90)
       (effects (font (size 1.27 1.27)) hide)
@@
     )
     (path "/29712cea-450e-4f0d-a15e-4194d0644920"
-      (reference "R3") (unit 1) (value "10k") (footprint "Resistor_SMD:R_0603_1608Metric_Pad0.98x0.95mm_HandSolder")
+      (reference "R3") (unit 1) (value "15k") (footprint "Resistor_SMD:R_0603_1608Metric_Pad0.98x0.95mm_HandSolder")
     )
     (path "/f3f8d0ad-904e-426e-97bd-00870b37ce69"
-      (reference "R4") (unit 1) (value "15k") (footprint "Resistor_SMD:R_0603_1608Metric_Pad0.98x0.95mm_HandSolder")
+      (reference "R4") (unit 1) (value "10k") (footprint "Resistor_SMD:R_0603_1608Metric_Pad0.98x0.95mm_HandSolder")
     )
     (path "/cdd3d6a2-e387-4601-8d8d-79ac383d8a86"

Commit message: Final tweaking and v1 gerber creation; JLC order placed
Parts:
- removed H1, H2: JLC_Tooling_Hole, Custom_Footprints:JLC_SMT_Tooling_Hole, symbol Mechanical:MountingHole
- added TP9: TestPoint, Custom_Footprints:1.3mm_Test_Point, symbol Connector:TestPoint
Connections:
- net GND: now also TP9.1
Other:
- moved on the sheet: FID1, J5, J6, TP1, TP2, TP3, TP4, TP5, TP6, TP7, TP8
