File: Hardware_v1_1/Punck_Components.kicad_pcb (KiCad board)
At the start: 4 copper layers, 91.2 x 100 mm, 114 parts, among them J1 Conn_01x12_Female, J2 Conn_01x12_Female, J3 Conn_01x12_Female, J4 Conn_01x12_Female, J5 Debug_Header, J6 SWD_Header, J7 Eurorack_10_pin_power, Q1 MMBT3904, Q2 MMBT3904, Q3 MMBT3904, Q4 MMBT3904, Q5 MMBT3904, Q6 MMBT3904, Q7 MMBT3904, U1 TL074, U2 STM32H743ZITx, U3 W25Q128JVS, U4 PCM5100APW, U5 W25Q128JVS, U6 TPS561201, U7 LD1117-3.3-4Tab, Y1 8MHz 20pF

Commit message: Updated crystal to 12 MHz
Parts:
- Y1: value 8MHz 20pF -> 12MHz 20pF
Changed lines of the file:
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@@
 			)
 		)
-		(property "Value" "8MHz 20pF"
+		(property "Value" "12MHz 20pF"
 			(at 0 2.8 0)
 			(layer "F.Fab")
